Commit message: Added gripper,camera to arm

File: open_manipulator_x_description/gazebo/open_manipulator_x.gazebo.xacro (robot description, xacro)
@@ -26,5 +26,5 @@
       <maxVel>1.0</maxVel>
       <minDepth>0.001</minDepth>
-      <material>Gazebo/DarkGrey</material>
+      <material>Gazebo/Gray</material>
     </gazebo>
   </xacro:macro>
@@ -36,7 +36,23 @@
   <xacro:Link reference="${prefix}gripper_left_link"/>
   <xacro:Link reference="${prefix}gripper_right_link"/>
-  <gazebo reference="${prefix}end_effector_link">
+  <gazebo reference="${prefix}gripper_left_link">
     <material>Gazebo/Red</material>
   </gazebo>
+  <gazebo reference="${prefix}gripper_right_link">
+    <material>Gazebo/Yellow</material>
+  </gazebo>
+<!--
+  <gazebo reference="${prefix}link1">
+    <material>Gazebo/Orange</material>
+  </gazebo>
+  <gazebo reference="${prefix}link2">
+    <material>Gazebo/Orange</material>
+  </gazebo>
+  <gazebo reference="${prefix}link3">
+    <material>Gazebo/Orange</material>
+  </gazebo>
+  <gazebo reference="${prefix}link4">
+    <material>Gazebo/Orange</material>
+  </gazebo> -->
   <xacro:SimpleTransmission trans="${prefix}trans1" joint="${prefix}joint1" actuator="${prefix}actuator1" />
   <xacro:SimpleTransmission trans="${prefix}trans2" joint="${prefix}joint2" actuator="${prefix}actuator2" />

File: open_manipulator_x_description/urdf/open_manipulator_x.urdf.xacro (robot description, xacro)
@@ -177,4 +177,31 @@
       </inertial>
     </link>
+    <joint name="${prefix}gripper_right_joint" type="fixed">
+      <parent link="${prefix}link5"/>
+      <child link="${prefix}gripper_right_link"/>
+      <origin xyz="0.09 0.0 0.0325" rpy="0 0 0 "/>
+    </joint>
+    <link name="${prefix}gripper_right_link">
+      <visual>
+        <origin xyz="0.0 0.0 0.0" rpy="-1.5708 0 -1.5708"/>
+        <geometry>
+          <mesh filename="${meshes_file_direction}/kkk.stl"/>
+        </geometry>
+        <material name="grey"/>
+      </visual>
+      <collision>
+        <origin xyz="0 0 0" rpy="-1.5708 0 -1.5708"/>
+        <geometry>
+          <mesh filename="${meshes_file_direction}/kkk.stl"/>
+        </geometry>
+      </collision>
+      <inertial>
+        <origin xyz="0 1.5708 0" />
+        <mass value="1.0e-03" />
+        <inertia ixx="1.0e-06" ixy="0.0" ixz="0.0"
+                 iyy="1.0e-06" iyz="0.0"
+                 izz="1.0e-06" />
+      </inertial>
+    </link>
     <joint name="${prefix}end_effector_joint" type="fixed">
       <parent link="${prefix}link5"/>
