Commit message: added camera plugins , removed gripper issues

File: open_manipulator_x_description/urdf/open_manipulator_x.urdf.xacro (robot description, xacro)
@@ -177,10 +177,12 @@
       </inertial>
     </link>
+    <xacro:intel_d435_camera prefix="${prefix}" parent_link="link5"/>
+<!--
     <joint name="${prefix}gripper_right_joint" type="fixed">
       <parent link="${prefix}link5"/>
-      <child link="${prefix}gripper_right_link"/>
+      <child link="${prefix}camera_link"/>
       <origin xyz="0.09 0.0 0.0325" rpy="0 0 0 "/>
     </joint>
-    <link name="${prefix}gripper_right_link">
+    <link name="${prefix}camera_link">
       <visual>
         <origin xyz="0.0 0.0 0.0" rpy="-1.5708 0 -1.5708"/>
@@ -203,11 +205,11 @@
                  izz="1.0e-06" />
       </inertial>
-    </link>
-    <joint name="${prefix}end_effector_joint" type="fixed">
+    </link> -->
+    <!-- <joint name="${prefix}end_effector_joint" type="fixed">
       <parent link="${prefix}link5"/>
       <child link="${prefix}end_effector_link"/>
       <origin xyz="0.123 0.0 0.0" rpy="0 0 0"/>
-    </joint>
-    <link name="${prefix}end_effector_link">
+    </joint> -->
+    <!-- <link name="${prefix}end_effector_link"> -->
       <!-- <visual>
         <origin xyz="0 0 0" rpy="0 0 0"/>
@@ -217,5 +219,5 @@
         <material name="red"/>
        </visual> -->
-    </link>
+    <!-- </link> -->
   </xacro:macro>
 </robot>

File: open_manipulator_x_description/urdf/open_manipulator_x_robot.urdf.xacro (robot description, xacro)
@@ -14,4 +14,5 @@
   <xacro:include filename="$(find open_manipulator_x_description)/urdf/open_manipulator_x.urdf.xacro" />
   <xacro:include filename="$(find open_manipulator_x_description)/ros2_control/open_manipulator_x_system.ros2_control.xacro" />
+  <xacro:include filename="$(find open_manipulator_x_description)/urdf/camera_module.urdf.xacro"/>
   <xacro:open_manipulator_x prefix="$(arg prefix)" />
   <xacro:open_manipulator_x_gazebo prefix="$(arg prefix)" />

File: open_manipulator_x_moveit_config/config/open_manipulator_x.ros2_control.xacro (robot description, xacro)
@@ -36,5 +36,5 @@
                 <state_interface name="velocity"/>
             </joint>
-            <joint name="gripper_left_joint">
+            <!-- <joint name="gripper_left_joint">
                 <command_interface name="position"/>
                 <state_interface name="position">
@@ -42,5 +42,5 @@
                 </state_interface>
                 <state_interface name="velocity"/>
-            </joint>
+            </joint> -->
         </ros2_control>
     </xacro:macro>
