Commit message: Changed teh depth position of point cloud,saved rviz config

File: open_manipulator_x_description/urdf/camera_module.urdf.xacro (robot description, xacro)
@@ -29,5 +29,16 @@
       <origin xyz="0.09 0.0 0.0325" rpy="0 0 0"/>
     </joint>
-    <!-- RGB Camera -->
+    <link name="${prefix}camera_depth_optical_frame"/>
+    <joint name="${prefix}camera_depth_optical_joint" type="fixed">
+      <parent link="${prefix}camera_link"/>
+      <child link="${prefix}camera_depth_optical_frame"/>
+      <origin xyz="0 0 0" rpy="-1.5708 0 -1.5708"/>
+    </joint>
+    <link name="${prefix}camera_rgb_optical_frame"/>
+    <joint name="${prefix}camera_rgb_optical_joint" type="fixed">
+      <parent link="${prefix}camera_link"/>
+      <child link="${prefix}camera_rgb_optical_frame"/>
+      <origin xyz="0 0 0" rpy="-1.5708 0 -1.5708"/>
+    </joint>
     <gazebo reference="${prefix}camera_link">
       <sensor name="d435_rgb" type="camera">
@@ -52,9 +63,8 @@
           <image_topic_name>image_raw</image_topic_name>
           <camera_info_topic_name>camera_info</camera_info_topic_name>
-          <frame_name>${prefix}camera_link</frame_name>
+          <frame_name>${prefix}camera_rgb_optical_frame</frame_name>
         </plugin>
       </sensor>
     </gazebo>
-    <!-- Infrared Cameras -->
     <gazebo reference="${prefix}camera_link">
       <sensor name="d435_infra1" type="camera">
@@ -79,5 +89,5 @@
           <image_topic_name>image_raw</image_topic_name>
           <camera_info_topic_name>camera_info</camera_info_topic_name>
-          <frame_name>${prefix}camera_link</frame_name>
+          <frame_name>${prefix}camera_depth_optical_frame</frame_name>
         </plugin>
       </sensor>
@@ -103,9 +113,8 @@
           <image_topic_name>image_raw</image_topic_name>
           <camera_info_topic_name>camera_info</camera_info_topic_name>
-          <frame_name>${prefix}camera_link</frame_name>
+          <frame_name>${prefix}camera_depth_optical_frame</frame_name>
         </plugin>
       </sensor>
     </gazebo>
-    <!-- Depth and Point Cloud Combined -->
     <gazebo reference="${prefix}camera_link">
       <sensor name="d435_depth" type="depth">
@@ -122,7 +131,4 @@
             <far>10.0</far>
           </clip>
-          <depth_camera>
-            <output>depth_and_point_cloud</output> <!-- THIS IS IMPORTANT -->
-          </depth_camera>
         </camera>
         <plugin name="${prefix}d435_depth_plugin" filename="libgazebo_ros_camera.so">
@@ -133,5 +139,5 @@
           <image_topic_name>image_raw</image_topic_name>
           <camera_info_topic_name>camera_info</camera_info_topic_name>
-          <frame_name>${prefix}camera_link</frame_name>
+          <frame_name>${prefix}camera_depth_optical_frame</frame_name>
         </plugin>
         <plugin name="${prefix}d435_pointcloud_plugin" filename="libgazebo_ros_point_cloud.so">
@@ -140,5 +146,5 @@
           </ros>
           <topic_name>points</topic_name>
-          <frame_name>${prefix}camera_link</frame_name>
+          <frame_name>${prefix}camera_depth_optical_frame</frame_name>
         </plugin>
       </sensor>
